File: _saved_LoRaNode.sch (KiCad schematic (older format))
At the start: 31 parts, among them J1 Conn_01x09, J2 Conn_01x03, J4 ISP, J5 Conn_01x06, J8 D2, J9 D3, SW1 SW_Push, U1 RFM95W-868S2, U4 ATMEGA328P-AU, Y1 8MHz HC5032/4

Commit message: Added LED, changed footprints to actual KiCAD library
Parts:
- U4: footprint Housings_QFP:TQFP-32_7x7mm_Pitch0.8mm -> Package_QFP:TQFP-32_7x7mm_P0.8mm
Changed lines of the file:
@@
 F 0 "U4" H 7475 4867 50  0000 C CNN
 F 1 "ATMEGA328P-AU" H 7475 4776 50  0000 C CNN
-F 2 "Housings_QFP:TQFP-32_7x7mm_Pitch0.8mm" H 7425 3500 50  0001 C CIN
+F 2 "Package_QFP:TQFP-32_7x7mm_P0.8mm" H 7425 3500 50  0001 C CIN
 F 3 "http://www.atmel.com/images/atmel-8271-8-bit-avr-microcontroller-atmega48a-48pa-88a-88pa-168a-168pa-328-328p_datasheet.pdf" H 7425 3500 50  0001 C CNN
 	1    7425 3500
